Commit message: Yo

File: src/test_chassis/urdf/test_chassis.urdf (robot description, URDF)
Before this commit: robot test_chassis, 7 links, 6 joints
Joints:
- joint base_to_wheel1: axis 0 0 0 -> 0 0 1; origin xyz=0.075 0.55 0.625 rpy=1.5708 1.5708 0 -> xyz=0 0 0 rpy=1.5708 1.5708 0
- joint base_to_wheel2: axis 0 0 0 -> 0 0 1
- joint base_to_wheel3: axis 0 0 0 -> 0 0 1
- joint base_to_wheel4: axis 0 0 0 -> 0 0 1
- joint base_to_wheel5: axis 0 0 0 -> 0 0 1
- joint base_to_wheel6: axis 0 0 0 -> 0 0 1
